Commit message: Gripper_correction

File: src/er_cobot_description/urdf/mycobot_280_urdf.xacro (robot description, xacro)
@@ -218,10 +218,10 @@
 		   		<mesh filename="file://$(find er_cobot_description)/meshes/mycobot_280/link7.dae"/>
 		  	</geometry>
-		  	<origin xyz = "0.0 0 -0.012 " rpy = "0 0 0"/>
+		  	<origin xyz = "0 0 -0.012 " rpy = "0 0 0"/>
 		</collision>
 	</link>
 	<link name="gripper_base">
 		<inertial>
-			<origin xyz="0 0 0.0" rpy="0 0 0"/>
+			<origin xyz="0.01 0.0 0.01" rpy="0 3.927 0"/>
 		  	<mass value="0.07"/>
 		  	<inertia
@@ -234,5 +234,5 @@
 				<mesh filename="file://$(find er_cobot_description)/meshes/mycobot_280/gripper_base.dae"/>
 		  	</geometry>
-		  	<origin xyz = "0.0 0.0 -0.012" rpy = "0 0 0"/>
+		  	<origin xyz = "0.01 0.0 0.01" rpy = "0 3.927 0"/>
 		</visual>
 		<collision>
@@ -240,10 +240,10 @@
 		   		<mesh filename="file://$(find er_cobot_description)/meshes/mycobot_280/gripper_base.dae"/>
 		  	</geometry>
-		  	<origin xyz = "0.0 0.0 -0.012" rpy = "0 0 0"/>
+		  	<origin xyz = "0.01 0.0 0.01" rpy = "0 3.927 0"/>
 		</collision>
 	</link>
 	<link name="gripper_left1">
 		<inertial>
-			<origin xyz="0 0 0.0" rpy="0 0 0"/>
+			<origin xyz="0.01 0 0.02" rpy="0 3.927 0"/>
 		  	<mass value="0.007"/>
 		  	<inertia
@@ -256,5 +256,5 @@
 		  		<mesh filename="file://$(find er_cobot_description)/meshes/mycobot_280/gripper_left1.dae"/>
 		  	</geometry>
-			<origin xyz = "0.039 -0.0133 -0.012 " rpy = " 0 0 0"/>
+			<origin xyz = "0.045 -0.0133 0.012 " rpy = " 0 3.927 0"/>
 		</visual>
 		<collision>
@@ -262,10 +262,10 @@
 		   		<mesh filename="file://$(find er_cobot_description)/meshes/mycobot_280/gripper_left1.dae"/>
 		  	</geometry>
-			<origin xyz = "0.039 -0.0133 -0.012 " rpy = " 0 0 0"/>
+			<origin xyz = "0.045 -0.0133 0.012 " rpy = " 0 3.927 0"/>
 		</collision>
 	</link>
 	<link name="gripper_left2">
 		<inertial>
-			<origin xyz="0 0 0.0" rpy="0 0 0"/>
+			<origin xyz="0 0 0.0" rpy="0 3.927 0"/>
 		  	<mass value="0.007"/>
 		  	<inertia
@@ -278,5 +278,5 @@
 		   		<mesh filename="file://$(find er_cobot_description)/meshes/mycobot_280/gripper_left2.dae"/>
 		  	</geometry>
-			<origin xyz = "0.005 -0.0195 -0.012 " rpy = " 0 0 0"/>
+			<origin xyz = "0.01 -0.0195 0.012 " rpy = " 0 3.927 0"/>
 		</visual>
 		<collision>
@@ -284,10 +284,10 @@
 		   		<mesh filename="file://$(find er_cobot_description)/meshes/mycobot_280/gripper_left2.dae"/>
 		  	</geometry>
-				<origin xyz = "0.005 -0.0195 -0.012 " rpy = " 0 0 0"/>
+				<origin xyz = "0.01 -0.0195 0.012 " rpy = " 0 3.927 0"/>
 		</collision>
 	</link>
 	<link name="gripper_left3">
 		<inertial>
-			<origin xyz="0 0 0.0" rpy="0 0 0"/>
+			<origin xyz="0 0 0.0" rpy = "0 3.927 0"/>
 		  	<mass value="0.007"/>
 		  	<inertia
@@ -300,5 +300,5 @@
 		   		<mesh filename="file://$(find er_cobot_description)/meshes/mycobot_280/gripper_left3.dae"/>
 		  	</geometry>
-		<origin xyz = "0.012 0.0025 -0.012 " rpy = " 0 0 0"/>
+		<origin xyz = "0.017 0.0025 0.012 " rpy = "0 3.927 0"/>
 		</visual>
 		<collision>
@@ -306,10 +306,10 @@
 		   		<mesh filename="file://$(find er_cobot_description)/meshes/mycobot_280/gripper_left3.dae"/>
 		  	</geometry>
-			<origin xyz = "0.012 0.0025 -0.012" rpy = " 0 0 0"/>
+			<origin xyz = "0.017 0.0025 0.012" rpy = "0 3.927 0"/>
 		</collision>
 	</link>
 	<link name="gripper_right1">
 		<inertial>
-			<origin xyz="0 0 0.0" rpy="0 0 0"/>
+			<origin xyz="0 0 0.0" rpy="0 3.927 0"/>
 		  	<mass value="0.007"/>
 		  	<inertia
@@ -322,5 +322,5 @@
 		   		<mesh filename="file://$(find er_cobot_description)/meshes/mycobot_280/gripper_right1.dae"/>
 		  	</geometry>
-			<origin xyz = "-0.039 -0.0133 -0.012 " rpy = " 0 0 0"/>
+			<origin xyz = "-0.03 -0.0133 0.006 " rpy = "0 3.927 0"/>
 		</visual>
 		<collision>
@@ -328,10 +328,10 @@
 		   		<mesh filename="file://$(find er_cobot_description)/meshes/mycobot_280/gripper_right1.dae"/>
 		  	</geometry>
-			<origin xyz = "-0.039 -0.0133 -0.012 " rpy = " 0 0 0"/>
+			<origin xyz = "-0.03 -0.0133 0.006 " rpy = "0 3.927 0"/>
 		</collision>
 	</link>
 	<link name="gripper_right2">
 		<inertial>
-			<origin xyz="0 0 0.0" rpy="0 0 0"/>
+			<origin xyz="0 0 0.0" rpy="0 3.927 0"/>
 		  	<mass value="0.007"/>
 		  	<inertia
@@ -344,5 +344,5 @@
 		   		<mesh filename="file://$(find er_cobot_description)/meshes/mycobot_280/gripper_right2.dae"/>
 		 	</geometry>
-			<origin xyz = "-0.005 -0.0195 -0.012 " rpy = " 0 0 0"/>
+			<origin xyz = "0.005 -0.0195 0.006 " rpy = "0 3.927 0"/>
 		</visual>
 		<collision>
@@ -350,10 +350,10 @@
 		   		<mesh filename="file://$(find er_cobot_description)/meshes/mycobot_280/gripper_right2.dae"/>
 		  	</geometry>
-			<origin xyz = "-0.005 -0.0195 -0.012 " rpy = " 0 0 0"/>
+			<origin xyz = "0.005 -0.0195 0.006 " rpy = "0 3.927 0"/>
 		</collision>
 	</link>
 	<link name="gripper_right3">
 		<inertial>
-			<origin xyz="0 0 0.0" rpy="0 0 0"/>
+			<origin xyz="0 0 0.0" rpy="0 3.927 0"/>
 		  	<mass value="0.007"/>
 		  	<inertia
@@ -366,5 +366,5 @@
 		   		<mesh filename="file://$(find er_cobot_description)/meshes/mycobot_280/gripper_right3.dae"/>
 			</geometry>
-			<origin xyz = "-0.012 0.0025 -0.012 " rpy = " 0 0 0"/>
+			<origin xyz = "0.005 0.0025 0.006 " rpy = "0 3.927 0"/>
 		</visual>
 		<collision>
@@ -372,5 +372,5 @@
 		   		<mesh filename="file://$(find er_cobot_description)/meshes/mycobot_280/gripper_right3.dae"/>
 		  	</geometry>
-			<origin xyz = "-0.012 0.0025 -0.012" rpy = " 0 0 0"/>
+			<origin xyz = "0.005 0.0025 0.006" rpy = "0 3.927 0"/>
 		</collision>
 	</link>
